File: stanislao_nrf.kicad_sch (KiCad schematic)
At the start: 19 parts, among them J1 Conn_01x06, Q1 BTS4140N, Q2 BSP89, U1 NRF52840-DONGLE, U2 LM5007MM

Commit message: Non chinese version
Parts:
- C2: footprint Capacitor_SMD:C_0402_1005Metric -> Capacitor_SMD:C_1206_3216Metric
- R1: footprint Resistor_SMD:R_0402_1005Metric -> Resistor_SMD:R_0603_1608Metric
Changed lines of the file:
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@@
   (junction (at 62.23 49.53) (diameter 1.016) (color 0 0 0 0))
   (junction (at 74.93 140.97) (diameter 1.016) (color 0 0 0 0))
-  (junction (at 76.2 151.13) (diameter 1.016) (color 0 0 0 0))
   (junction (at 80.01 140.97) (diameter 1.016) (color 0 0 0 0))
   (junction (at 80.01 146.05) (diameter 1.016) (color 0 0 0 0))
@@
     (stroke (width 0) (type solid) (color 0 0 0 0))
   )
-  (wire (pts (xy 94.234 140.97) (xy 94.234 140.97))
-    (stroke (width 0) (type solid) (color 0 0 0 0))
-  )
   (wire (pts (xy 94.234 140.97) (xy 100.33 140.97))
     (stroke (width 0) (type solid) (color 0 0 0 0))
@@
     (property "Reference" "R1" (id 0) (at 45.72 138.5632 90))
     (property "Value" "127K" (id 1) (at 45.72 140.862 90))
-    (property "Footprint" "Resistor_SMD:R_0402_1005Metric" (id 2) (at 45.72 135.89 0)
+    (property "Footprint" "Resistor_SMD:R_0603_1608Metric" (id 2) (at 45.72 135.89 0)
       (effects (font (size 1.27 1.27)) hide)
     )
@@
       (effects (font (size 1.27 1.27)) (justify left))
     )
-    (property "Footprint" "Capacitor_SMD:C_0402_1005Metric" (id 2) (at 31.75 135.89 0)
+    (property "Footprint" "Capacitor_SMD:C_1206_3216Metric" (id 2) (at 31.75 135.89 0)
       (effects (font (size 1.27 1.27)) hide)
     )
@@
     )
     (path "/f08c29ff-7b24-4c45-a79d-9bc796a15712"
-      (reference "C2") (unit 1) (value "0.1uF") (footprint "Capacitor_SMD:C_0402_1005Metric")
+      (reference "C2") (unit 1) (value "0.1uF") (footprint "Capacitor_SMD:C_1206_3216Metric")
     )
     (path "/6be3c013-4e81-42b7-b5e9-5dd302254d07"
@@
     )
     (path "/eeb54523-614c-4001-a285-cf6390986c44"
-      (reference "R1") (unit 1) (value "127K") (footprint "Resistor_SMD:R_0402_1005Metric")
+      (reference "R1") (unit 1) (value "127K") (footprint "Resistor_SMD:R_0603_1608Metric")
     )
     (path "/63411555-c8ea-41d5-be90-4536d193ce54"

Commit message: Cleanup
Parts:
- added Q?: BSP89, Package_TO_SOT_SMD:SOT-223-3_TabPin2, symbol Transistor_FET:BSP89
- added Q?: BTS4140N, Package_TO_SOT_SMD:SOT-223-3_TabPin2, symbol Transistor_FET:BSP89
- added R? (x4): R_Small, symbol Device:R_Small
- J1: value Conn_01x06 -> JST_HX_S6B
Connections:
- net BTS414ON_CTRL: no longer Q1.1 (G), Q2.2 (D)
- net GND: now also J1.6 (Pin_6), Q?.3 (S); no longer J1.1 (Pin_1)
- net P1.00: now also R?.2, R?.2; no longer Q2.1 (G)
- net TSDZ2_BRAKE_INPUT: now also J1.5 (Pin_5); no longer J1.2 (Pin_2)
- net TSDZ2_RX: now also J1.4 (Pin_4); no longer J1.3 (Pin_3)
- net TSDZ2_TX: now also J1.2 (Pin_2); no longer J1.5 (Pin_5)
- net TSDZ2_VIN: now also J1.1 (Pin_1), Q?.3 (S); no longer J1.6 (Pin_6)
- net VBUS: now reaches C6.1, C7.2, L1.2, R3.1, U1.VBUS
- net V_BATT renamed +VDC
- net +VDC: now also J1.3 (Pin_3), Q?.2 (D), R?.1, R?.1; no longer J1.4 (Pin_4)
- new net: Q?.1 (G), R?.1
- new net: Q?.1 (G), Q?.2 (D), R?.2
- new net: Q1.1 (G), Q2.2 (D), R?.2
- new net: Q2.1 (G), R?.1
Other:
- moved on the sheet: C1, C2, C3, C4, C5, C6, C7, D1, J1, L1, Q1, Q2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

Commit message: Smol dc/dc
Parts:
- removed C2: 0.1uF, Capacitor_SMD:C_1206_3216Metric, symbol Device:C_Small
- removed C3, C4, C5: 0.1uF, Capacitor_SMD:C_0402_1005Metric, symbol Device:C_Small
- removed C7: 3nF, Capacitor_SMD:C_0402_1005Metric, symbol Device:C_Small
- removed D1: D_Schottky_Small, Diode_SMD:D_SOD-123F, symbol Device:D_Schottky_Small
- removed L1: 100uH, Inductor_SMD:L_TracoPower_TCK-047_5.2x5.8mm, symbol Device:L_Small
- removed Q?: BSP89, Package_TO_SOT_SMD:SOT-223-3_TabPin2, symbol Transistor_FET:BSP89
- removed Q?: BTS4140N, Package_TO_SOT_SMD:SOT-223-3_TabPin2, symbol Transistor_FET:BSP89
- removed R2: 278K, Resistor_SMD:R_0402_1005Metric, symbol Device:R_Small
- removed R3, R4: 1K, Resistor_SMD:R_0402_1005Metric, symbol Device:R_Small
- removed R5: 100K, Resistor_SMD:R_0402_1005Metric, symbol Device:R_Small
- removed R? (x3): R_Small, symbol Device:R_Small
- removed U2: LM5007MM, Package_SO:MSOP-8_3x3mm_P0.65mm, symbol Regulator_Switching:LM5007MM
- added J2, J3, J4, J5: Conn_01x02, Connector_JST:JST_XH_B2B-XH-A_1x02_P2.50mm_Vertical, symbol Connector_Generic:Conn_01x02
- added U2: TPSM265R1, stanislao_nrf-backups:TPSM265R1, symbol stanislao_nrf:TPSM265R1
- C1: value 10uF -> 2.2uF
- C6: value 10uF -> 22uF
- R1: value 127K -> R_Small
- R6: renamed from R?; footprint (none) -> Resistor_SMD:R_0603_1608Metric
Connections:
- net GND: now also J1.1 (Pin_1), U2.11 (GND), U2.3 (GND), U2.6 (GND); no longer J1.6 (Pin_6)
- net P1.00: now also R1.2
- net TSDZ2_BRAKE_INPUT: now also J1.2 (Pin_2); no longer J1.5 (Pin_5)
- net TSDZ2_RX: now also J1.3 (Pin_3); no longer J1.4 (Pin_4)
- net TSDZ2_TX: now also J1.5 (Pin_5); no longer J1.2 (Pin_2)
- net TSDZ2_VIN: now also J1.6 (Pin_6); no longer J1.1 (Pin_1)
- net VBUS: now also U2.1 (VOUT), U2.8 (FB)
- net at Q2.1 (G): now also R1.1
- net +VDC renamed V_BATT
- net V_BATT: now also J1.4 (Pin_4), U2.4 (VIN), U2.5 (VIN), U2.9 (EN); no longer J1.3 (Pin_3), R1.1
- no-connect marks 14 -> 17
Other:
- moved on the sheet: C6, J1

Commit message: Awaiting for logo
Parts:
- removed J2, J3, J4, J5: Conn_01x02, Connector_JST:JST_XH_B2B-XH-A_1x02_P2.50mm_Vertical, symbol Connector_Generic:Conn_01x02
- removed Q1: BTS4140N, Package_TO_SOT_SMD:SOT-223-3_TabPin2, symbol Transistor_FET:BSP89
- removed Q2: BSP89, Package_TO_SOT_SMD:SOT-223-3_TabPin2, symbol Transistor_FET:BSP89
- removed R1: R_Small, Resistor_SMD:R_0603_1608Metric, symbol Device:R_Small
- added Q1: SSM6J507NU, footprints:UDFN6B, symbol SSM6J507NU:SSM6J507NU
- added SW1, SW2, SW3, SW4: SW_Push, Connector_JST:JST_XH_B2B-XH-A_1x02_P2.50mm_Vertical, symbol Switch:SW_Push
- R6: value R_Small -> DNP/100KOhm
Connections:
- net GND: now also R6.2, SW1.1, SW2.1, SW3.1, SW4.1
- net TSDZ2_VIN: now also Q1.4 (S), Q1.S
- net V_BATT: now also Q1.1 (D), Q1.2 (D), Q1.5 (D), Q1.6 (D), Q1.D; no longer R6.1
- net P0.13_UP: now reaches U1.0.13
- net P0.13_UP: now also SW1.2
- net P0.15_ENTER: now reaches U1.0.15
- net P0.15_ENTER: now also SW3.2
- net P0.17_DOWN: now reaches U1.0.17
- net P0.17_DOWN: now also SW2.2
- net P0.20_POWER: now reaches U1.0.20
- net P0.20_POWER: now also SW4.2
- net P1.00 renamed P1.00_VIN_CTRL
- net P1.00_VIN_CTRL: now also R6.1, Q1.3 (G)
- no-connect marks 17 -> 13
Other:
- moved on the sheet: C1, C6, J1, R6, U1, U2
